File: hardware/main_pcb/cpu.kicad_sch (KiCad schematic)
At the start: 28 parts

Commit message: - Initial PCB layout
Parts:
- C1, C11, C14, C2, C3, C4, C5, C6, C7, C9: renamed from C?; value 100n -> 100nF
- C10, C8: value 1u -> 1uF
- SW1: renamed from SW?; value SW_Push -> SKQG; footprint (none) -> Button_Switch_SMD:SW_SPST_SKQG_WithStem
- gave numbers to parts that had none: 13
- renumbered MCU_JTAG to MCU_JTAG1
Connections:
- net RESET renamed RUN
