File: hardware/main_pcb/keypad.kicad_sch (KiCad schematic)
At the start: 2 parts, among them J400 Conn_01x05, J401 Conn_01x05

Commit message: - Initial PCB layout
Parts:
- removed J400, J401: Conn_01x05, symbol Connector_Generic:Conn_01x05
- added J400, J401, J402: Conn_01x03, Connector_PinHeader_1.27mm:PinHeader_1x03_P1.27mm_Vertical, symbol Connector_Generic:Conn_01x03
- added SW400, SW401: SKQG, Button_Switch_SMD:SW_SPST_SKQG_WithStem, symbol Switch:SW_Push
Connections:
- net +3V3: now also J401.1 (Pin_1)
- net +BATT: now also J402.1 (Pin_1)
- net BAT_NTC: now also J402.2 (Pin_2)
- net GND: now also J400.3 (Pin_3), J402.3 (Pin_3), SW400.2, SW401.2
- net KP_KEY1: now also J401.2 (Pin_2), SW400.1
- net KP_KEY2: now also J401.3 (Pin_3), SW401.1
- net KP_SCL: now also J400.1 (Pin_1)
- net KP_SDA: now also J400.2 (Pin_2)
- no-connect marks 1 -> 0
