File: hardware/main_pcb/storage.kicad_sch (KiCad schematic)
At the start: 12 parts, among them J300 MICRO_SD(TFC-WPAPR-08), U300 NX3P1108UK

Commit message: - Initial PCB layout
Parts:
- removed R300: 47K, Resistor_SMD:R_0402_1005Metric, symbol Device:R
- U300: footprint (none) -> Package_CSP:WLCSP-4-X1-WLB0909-4_0.89x0.89mm_P0.5mm
Changed lines of the file:
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@@
   (junction (at 172.72 81.28) (diameter 0.9144) (color 0 0 0 0))
   (junction (at 172.72 88.9) (diameter 0.9144) (color 0 0 0 0))
-  (junction (at 182.88 81.28) (diameter 0.9144) (color 0 0 0 0))
-  (junction (at 182.88 88.9) (diameter 0.9144) (color 0 0 0 0))
   (wire (pts (xy 99.06 71.12) (xy 121.92 71.12))
     (stroke (width 0) (type solid) (color 0 0 0 0))
@@
     (stroke (width 0) (type solid) (color 0 0 0 0))
   )
-  (wire (pts (xy 182.88 81.28) (xy 193.04 81.28))
-    (stroke (width 0) (type solid) (color 0 0 0 0))
-  )
   (wire (pts (xy 182.88 88.9) (xy 172.72 88.9))
     (stroke (width 0) (type solid) (color 0 0 0 0))
   )
-  (wire (pts (xy 182.88 88.9) (xy 193.04 88.9))
-    (stroke (width 0) (type solid) (color 0 0 0 0))
-  )
   (text "47uF is required to comply with SD 3.0 spec" (at 177.8 91.44 0)
     (effects (font (size 1.27 1.27)) (justify left bottom))
@@
   (symbol (lib_id "power:+3V3") (at 119.38 63.5 0) (unit 1)
     (in_bom yes) (on_board yes)
-    (property "Reference" "#PWR?" (id 0) (at 119.38 67.31 0)
+    (property "Reference" "#PWR041" (id 0) (at 119.38 67.31 0)
       (effects (font (size 1.27 1.27)) hide)
     )
@@
   (symbol (lib_id "symbols:+VSD") (at 144.78 63.5 0) (unit 1)
     (in_bom yes) (on_board yes)
-    (property "Reference" "#PWR?" (id 0) (at 144.78 67.31 0)
+    (property "Reference" "#PWR043" (id 0) (at 144.78 67.31 0)
       (effects (font (size 1.27 1.27)) hide)
     )
@@
   (symbol (lib_id "power:GND") (at 139.7 71.12 0) (unit 1)
     (in_bom yes) (on_board yes)
-    (property "Reference" "#PWR?" (id 0) (at 139.7 77.47 0)
+    (property "Reference" "#PWR042" (id 0) (at 139.7 77.47 0)
       (effects (font (size 1.27 1.27)) hide)
     )
@@
     (pin "2")
   )
-  (symbol (lib_id "Device:R") (at 193.04 85.09 0) (unit 1)
-    (in_bom yes) (on_board yes)
-    (property "Reference" "R300" (id 0) (at 194.818 83.922 0)
-      (effects (font (size 1.27 1.27)) (justify left))
-    )
-    (property "Value" "47K" (id 1) (at 194.818 86.233 0)
-      (effects (font (size 1.27 1.27)) (justify left))
-    )
-    (property "Footprint" "Resistor_SMD:R_0402_1005Metric" (id 2) (at 191.262 85.09 90)
-      (effects (font (size 1.27 1.27)) hide)
-    )
-    (property "Datasheet" "~" (id 3) (at 193.04 85.09 0)
-      (effects (font (size 1.27 1.27)) hide)
-    )
-    (pin "1")
-    (pin "2")
-  )
   (symbol (lib_id "Device:C") (at 154.94 123.19 0) (unit 1)
     (in_bom yes) (on_board yes)
@@
     (property "Reference" "U300" (id 0) (at 129.54 58.42 0))
     (property "Value" "NX3P1108UK" (id 1) (at 129.54 60.96 0))
-    (property "Footprint" "" (id 2) (at 129.54 58.42 0)
-      (effects (font (size 1.27 1.27)) hide)
-    )
+    (property "Footprint" "Package_CSP:WLCSP-4-X1-WLB0909-4_0.89x0.89mm_P0.5mm" (id 2) (at 129.54 58.42 0)
+      (effects (font (size 1.27 1.27)) hide)
+    )
