File: hardware/main_pcb/usb.kicad_sch (KiCad schematic)
At the start: 8 parts, among them U200 NX5P2090, U201 NX18P3001

Commit message: - Initial PCB layout
Parts:
- J1: renamed from J?; footprint (none) -> Connector_USB:USB_Micro-AB_Molex_47590-0001
Connections:
- net USB_DM: now also U201.D3 (ID); no longer U201.D1 (D-)
- net USB_ID: now also U201.D1 (D-); no longer U201.D3 (ID)
Changed lines of the file:
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@@
   (junction (at 144.78 99.06) (diameter 0.9144) (color 0 0 0 0))
   (junction (at 144.78 101.6) (diameter 0.9144) (color 0 0 0 0))
-  (junction (at 154.94 111.76) (diameter 0.9144) (color 0 0 0 0))
+  (junction (at 154.94 109.22) (diameter 0.9144) (color 0 0 0 0))
   (junction (at 157.48 106.68) (diameter 0.9144) (color 0 0 0 0))
-  (junction (at 160.02 109.22) (diameter 0.9144) (color 0 0 0 0))
+  (junction (at 160.02 111.76) (diameter 0.9144) (color 0 0 0 0))
   (junction (at 162.56 50.8) (diameter 0.9144) (color 0 0 0 0))
   (junction (at 162.56 83.82) (diameter 0.9144) (color 0 0 0 0))
@@
     (stroke (width 0) (type solid) (color 0 0 0 0))
   )
-  (wire (pts (xy 127 109.22) (xy 160.02 109.22))
-    (stroke (width 0) (type solid) (color 0 0 0 0))
-  )
-  (wire (pts (xy 127 111.76) (xy 154.94 111.76))
+  (wire (pts (xy 127 109.22) (xy 154.94 109.22))
+    (stroke (width 0) (type solid) (color 0 0 0 0))
+  )
+  (wire (pts (xy 127 111.76) (xy 160.02 111.76))
     (stroke (width 0) (type solid) (color 0 0 0 0))
   )
@@
     (stroke (width 0) (type solid) (color 0 0 0 0))
   )
-  (wire (pts (xy 154.94 91.44) (xy 154.94 111.76))
-    (stroke (width 0) (type solid) (color 0 0 0 0))
-  )
-  (wire (pts (xy 154.94 111.76) (xy 165.1 111.76))
+  (wire (pts (xy 154.94 91.44) (xy 154.94 109.22))
+    (stroke (width 0) (type solid) (color 0 0 0 0))
+  )
+  (wire (pts (xy 154.94 109.22) (xy 165.1 109.22))
     (stroke (width 0) (type solid) (color 0 0 0 0))
   )
@@
     (stroke (width 0) (type solid) (color 0 0 0 0))
   )
-  (wire (pts (xy 160.02 86.36) (xy 160.02 109.22))
-    (stroke (width 0) (type solid) (color 0 0 0 0))
-  )
-  (wire (pts (xy 160.02 109.22) (xy 165.1 109.22))
+  (wire (pts (xy 160.02 86.36) (xy 160.02 111.76))
+    (stroke (width 0) (type solid) (color 0 0 0 0))
+  )
+  (wire (pts (xy 160.02 111.76) (xy 165.1 111.76))
     (stroke (width 0) (type solid) (color 0 0 0 0))
   )
@@
   (symbol (lib_id "power:GND") (at 132.08 71.12 0) (mirror y) (unit 1)
     (in_bom yes) (on_board yes)
-    (property "Reference" "#PWR?" (id 0) (at 132.08 77.47 0)
+    (property "Reference" "#PWR076" (id 0) (at 132.08 77.47 0)
       (effects (font (size 1.27 1.27)) hide)
     )
@@
   (symbol (lib_id "power:GND") (at 144.78 68.58 0) (mirror y) (unit 1)
     (in_bom yes) (on_board yes)
-    (property "Reference" "#PWR?" (id 0) (at 144.78 74.93 0)
+    (property "Reference" "#PWR077" (id 0) (at 144.78 74.93 0)
       (effects (font (size 1.27 1.27)) hide)
     )
@@
   (symbol (lib_id "power:GND") (at 144.78 101.6 0) (mirror y) (unit 1)
     (in_bom yes) (on_board yes)
-    (property "Reference" "#PWR?" (id 0) (at 144.78 107.95 0)
+    (property "Reference" "#PWR078" (id 0) (at 144.78 107.95 0)
       (effects (font (size 1.27 1.27)) hide)
     )
@@
   (symbol (lib_id "power:GND") (at 170.18 58.42 0) (mirror y) (unit 1)
     (in_bom yes) (on_board yes)
-    (property "Reference" "#PWR?" (id 0) (at 170.18 64.77 0)
+    (property "Reference" "#PWR079" (id 0) (at 170.18 64.77 0)
       (effects (font (size 1.27 1.27)) hide)
     )
@@
   (symbol (lib_id "Connector:USB_B_Micro") (at 172.72 106.68 0) (mirror y) (unit 1)
     (in_bom yes) (on_board yes)
-    (property "Reference" "J?" (id 0) (at 179.07 107.95 0)
+    (property "Reference" "J1" (id 0) (at 179.07 107.95 0)
       (effects (font (size 1.27 1.27)) (justify right))
     )
@@
       (effects (font (size 1.27 1.27)) (justify right))
     )
-    (property "Footprint" "" (id 2) (at 168.91 107.95 0)
-      (effects (font (size 1.27 1.27)) hide)
-    )
+    (property "Footprint" "Connector_USB:USB_Micro-AB_Molex_47590-0001" (id 2) (at 168.91 107.95 0)
+      (effects (font (size 1.27 1.27)) hide)
+    )
