File: hardware/main_pcb/lcd.kicad_sch (KiCad schematic)
At the start: 47 parts, among them J500 Conn_01x24_MountingPin, U500 DS4424, U501 NX3P1108UK, U502 LT1615, U503 MIC5233YM5, U504 MIC5233YM5, U505 MIC5233YM5, U506 MIC5233YM5

Commit message: - Initial PCB layout
Parts:
- removed C505: 22uF/50V, Capacitor_SMD:C_1206_3216Metric, symbol Device:C
- C500: footprint Capacitor_SMD:C_0603_1608Metric -> Capacitor_SMD:C_0402_1005Metric
- C502: value 220nF -> 1uF; footprint Capacitor_SMD:C_0603_1608Metric -> Capacitor_SMD:C_0402_1005Metric
- C506, C507, C508, C509, C510, C511, C512, C513, C514: footprint Capacitor_SMD:C_0603_1608Metric -> Capacitor_SMD:C_0805_2012Metric
- C515: value 220nF -> 100nF; footprint Capacitor_SMD:C_0603_1608Metric -> Capacitor_SMD:C_0402_1005Metric
- R500, R501, R502, R503, R504, R505, R506, R507, R508, R509, R510, R511, R512, R513, R514, R515, R516, R517: footprint Resistor_SMD:R_0603_1608Metric -> Resistor_SMD:R_0402_1005Metric
- U501: footprint (none) -> Package_CSP:WLCSP-4-X1-WLB0909-4_0.89x0.89mm_P0.5mm
Connections:
- net LCD_COMLP: now also RN500.8 (R1.2); no longer RN500.1 (R1.1)
- net LCD_D0: now also RN502.5 (R4.2); no longer RN502.4 (R4.1)
- net LCD_D1: now also RN502.6 (R3.2); no longer RN502.3 (R3.1)
- net LCD_D2: now also RN502.7 (R2.2); no longer RN502.2 (R2.1)
- net LCD_D3: now also RN502.8 (R1.2); no longer RN502.1 (R1.1)
- net LCD_D4: now also RN501.5 (R4.2); no longer RN501.4 (R4.1)
- net LCD_D5: now also RN501.6 (R3.2); no longer RN501.3 (R3.1)
- net LCD_D6: now also RN501.7 (R2.2); no longer RN501.2 (R2.1)
- net LCD_D7: now also RN501.8 (R1.2); no longer RN501.1 (R1.1)
- net LCD_FLM: now also RN500.7 (R2.2); no longer RN500.2 (R2.1)
- net LCD_M: now also RN500.6 (R3.2); no longer RN500.3 (R3.1)
- net LCD_SEGLP: now also RN500.5 (R4.2); no longer RN500.4 (R4.1)
- net at J500.11 (Pin_11): now also RN500.4 (R4.1); no longer RN500.5 (R4.2)
- net at J500.9 (Pin_9): now also RN500.3 (R3.1); no longer RN500.6 (R3.2)
- net at J500.8 (Pin_8): now also RN500.2 (R2.1); no longer RN500.7 (R2.2)
- net at J500.6 (Pin_6): now also RN500.1 (R1.1); no longer RN500.8 (R1.2)
- net at J500.16 (Pin_16): now also RN501.1 (R1.1); no longer RN501.8 (R1.2)
- net at J500.17 (Pin_17): now also RN501.2 (R2.1); no longer RN501.7 (R2.2)
- net at J500.18 (Pin_18): now also RN501.3 (R3.1); no longer RN501.6 (R3.2)
- net at J500.19 (Pin_19): now also RN501.4 (R4.1); no longer RN501.5 (R4.2)
- net at J500.20 (Pin_20): now also RN502.1 (R1.1); no longer RN502.8 (R1.2)
- net at J500.21 (Pin_21): now also RN502.2 (R2.1); no longer RN502.7 (R2.2)
- net at J500.22 (Pin_22): now also RN502.3 (R3.1); no longer RN502.6 (R3.2)
- net at J500.23 (Pin_23): now also RN502.4 (R4.1); no longer RN502.5 (R4.2)
Other:
- note removed: "I2C Address: 0b0010000"
- moved on the sheet: RN500, RN501, RN502

Commit message: - PCB rev 0p1 draft
Connections:
- net LCD_D0: now also RN501.8 (R1.2); no longer RN502.5 (R4.2)
- net LCD_D1: now also RN501.7 (R2.2); no longer RN502.6 (R3.2)
- net LCD_D2: now also RN501.6 (R3.2); no longer RN502.7 (R2.2)
- net LCD_D3: now also RN501.5 (R4.2); no longer RN502.8 (R1.2)
- net LCD_D4: now also RN502.8 (R1.2); no longer RN501.5 (R4.2)
- net LCD_D5: now also RN502.7 (R2.2); no longer RN501.6 (R3.2)
- net LCD_D6: now also RN502.6 (R3.2); no longer RN501.7 (R2.2)
- net LCD_D7: now also RN502.5 (R4.2); no longer RN501.8 (R1.2)
Changed lines of the file:
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@@
     (effects (font (size 1.27 1.27)) (justify right))
   )
-  (hierarchical_label "LCD_D7" (shape input) (at 205.74 109.22 180)
+  (hierarchical_label "LCD_D0" (shape input) (at 205.74 109.22 180)
     (effects (font (size 1.27 1.27)) (justify right))
   )
-  (hierarchical_label "LCD_D6" (shape input) (at 205.74 111.76 180)
+  (hierarchical_label "LCD_D1" (shape input) (at 205.74 111.76 180)
     (effects (font (size 1.27 1.27)) (justify right))
   )
-  (hierarchical_label "LCD_D5" (shape input) (at 205.74 114.3 180)
+  (hierarchical_label "LCD_D2" (shape input) (at 205.74 114.3 180)
     (effects (font (size 1.27 1.27)) (justify right))
   )
-  (hierarchical_label "LCD_D4" (shape input) (at 205.74 116.84 180)
+  (hierarchical_label "LCD_D3" (shape input) (at 205.74 116.84 180)
     (effects (font (size 1.27 1.27)) (justify right))
   )
-  (hierarchical_label "LCD_D3" (shape input) (at 205.74 119.38 180)
+  (hierarchical_label "LCD_D4" (shape input) (at 205.74 119.38 180)
     (effects (font (size 1.27 1.27)) (justify right))
   )
-  (hierarchical_label "LCD_D2" (shape input) (at 205.74 121.92 180)
+  (hierarchical_label "LCD_D5" (shape input) (at 205.74 121.92 180)
     (effects (font (size 1.27 1.27)) (justify right))
   )
-  (hierarchical_label "LCD_D1" (shape input) (at 205.74 124.46 180)
+  (hierarchical_label "LCD_D6" (shape input) (at 205.74 124.46 180)
     (effects (font (size 1.27 1.27)) (justify right))
   )
-  (hierarchical_label "LCD_D0" (shape input) (at 205.74 127 180)
+  (hierarchical_label "LCD_D7" (shape input) (at 205.74 127 180)
     (effects (font (size 1.27 1.27)) (justify right))
   )
