File: hardware/main_pcb/pcb.kicad_sch (KiCad schematic)
At the start: 0 parts

Commit message: - Initial PCB layout
Other:
- sheet cpu ports: added none; removed RESET
- sheet power ports: added none; removed SYS_RESET
- note added: "I2C Address: 0b0010000"
- note added: "I2C Address: 0b0010100"
- note added: "I2C Address: 0b1011010"

Commit message: - PCB rev 0p1 draft
Changed lines of the file:
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@@
       (effects (font (size 1.27 1.27)) (justify left))
     )
-    (pin "LCD_DISPON" input (at 137.16 116.84 180)
-      (effects (font (size 1.27 1.27)) (justify left))
-    )
-    (pin "LCD_SEGLP" input (at 137.16 119.38 180)
+    (pin "LCD_DISPON" input (at 137.16 127 180)
+      (effects (font (size 1.27 1.27)) (justify left))
+    )
+    (pin "LCD_SEGLP" input (at 137.16 124.46 180)
       (effects (font (size 1.27 1.27)) (justify left))
     )
@@
       (effects (font (size 1.27 1.27)) (justify left))
     )
-    (pin "LCD_CP" input (at 137.16 124.46 180)
+    (pin "LCD_CP" input (at 137.16 129.54 180)
       (effects (font (size 1.27 1.27)) (justify left))
     )
@@
       (effects (font (size 1.27 1.27)) (justify left))
     )
-    (pin "LCD_COMLP" input (at 137.16 127 180)
-      (effects (font (size 1.27 1.27)) (justify left))
-    )
-    (pin "LCD_FLM" input (at 137.16 129.54 180)
+    (pin "LCD_COMLP" input (at 137.16 116.84 180)
+      (effects (font (size 1.27 1.27)) (justify left))
+    )
+    (pin "LCD_FLM" input (at 137.16 119.38 180)
       (effects (font (size 1.27 1.27)) (justify left))
     )
@@
       (reference "#PWR015") (unit 1) (value "GND") (footprint "")
     )
-    (path "/00000000-0000-0000-0000-00005d4c99f9/ca59aaa1-81c4-4ac1-8fb0-99adef2834d5"
-      (reference "#PWR016") (unit 1) (value "GND") (footprint "")
-    )
     (path "/00000000-0000-0000-0000-00005d4c99f9/e92868d4-2392-4126-a8ce-1e6fb38e9cbc"
       (reference "#PWR017") (unit 1) (value "GND") (footprint "")
@@
       (reference "L101") (unit 1) (value "4.7uH") (footprint "Inductor_SMD:L_Vishay_IHLP-1212")
     )
-    (path "/00000000-0000-0000-0000-00005d4c99f9/87fa8bc4-ce71-43c0-a610-0c15c47fac56"
-      (reference "R101") (unit 1) (value "100K/1%") (footprint "Resistor_SMD:R_0402_1005Metric")
-    )
     (path "/00000000-0000-0000-0000-00005d4c99f9/df375d3c-7eff-4aaf-9a0f-d92f216bb3ae"
