File: hardware/main_pcb/power.kicad_sch (KiCad schematic)
At the start: 15 parts, among them SW100 SW_Push, U100 ADP5360

Commit message: - Initial PCB layout
Parts:
- removed R100, R102: 10K, Resistor_SMD:R_0603_1608Metric, symbol Device:R
- removed SW100: SW_Push, symbol Switch:SW_Push
- C103: footprint Capacitor_SMD:C_0603_1608Metric -> Capacitor_SMD:C_0402_1005Metric
- R101: footprint Resistor_SMD:R_0603_1608Metric -> Resistor_SMD:R_0402_1005Metric
- U100: footprint (none) -> footprints:WLCSP-32_6x6_2.56x2.56mm
Connections:
- net +SYS: now also U100.E2 (EN1)
- net +5V renamed VBUS_OTG
- net SYS_RESET: no longer names the net of U100.E3 (~RESET)
- no-connect marks 4 -> 6

Commit message: - PCB rev 0p1 draft
Parts:
- removed R101: 100K/1%, Resistor_SMD:R_0402_1005Metric, symbol Device:R
Connections:
- no-connect marks 6 -> 7
Other:
- note added: "Note: After powering up, the output is by default 1.8V, need to be set to 3.3V using software"
Changed lines of the file:
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@@
   (no_connect (at 106.68 127))
   (no_connect (at 106.68 129.54))
+  (no_connect (at 137.16 96.52))
   (no_connect (at 137.16 127))
   (no_connect (at 137.16 129.54))
@@
     (stroke (width 0) (type solid) (color 0 0 0 0))
   )
-  (wire (pts (xy 137.16 96.52) (xy 142.24 96.52))
-    (stroke (width 0) (type solid) (color 0 0 0 0))
-  )
   (wire (pts (xy 137.16 101.6) (xy 152.4 101.6))
     (stroke (width 0) (type solid) (color 0 0 0 0))
@@
   )
   (wire (pts (xy 149.86 73.66) (xy 152.4 73.66))
-    (stroke (width 0) (type solid) (color 0 0 0 0))
-  )
-  (wire (pts (xy 149.86 96.52) (xy 152.4 96.52))
     (stroke (width 0) (type solid) (color 0 0 0 0))
   )
@@
   (text "Combined capacitance for VBUS and VDD must not exceed 10uF"
     (at 88.9 60.96 0)
+    (effects (font (size 1.27 1.27)) (justify left bottom))
+  )
+  (text "Note: After powering up, the output is by default 1.8V, need to be set to 3.3V using software"
+    (at 142.24 99.06 0)
     (effects (font (size 1.27 1.27)) (justify left bottom))
   )
@@
     (pin "1")
   )
-  (symbol (lib_id "power:GND") (at 152.4 96.52 90) (mirror x) (unit 1)
-    (in_bom yes) (on_board yes)
-    (property "Reference" "#PWR016" (id 0) (at 158.75 96.52 0)
-      (effects (font (size 1.27 1.27)) hide)
-    )
-    (property "Value" "GND" (id 1) (at 158.0642 96.647 90))
-    (property "Footprint" "" (id 2) (at 152.4 96.52 0)
-      (effects (font (size 1.27 1.27)) hide)
-    )
-    (property "Datasheet" "" (id 3) (at 152.4 96.52 0)
-      (effects (font (size 1.27 1.27)) hide)
-    )
-    (pin "1")
-  )
   (symbol (lib_id "power:GND") (at 152.4 101.6 90) (mirror x) (unit 1)
     (in_bom yes) (on_board yes)
@@
     (pin "1")
   )
-  (symbol (lib_id "Device:R") (at 146.05 96.52 90) (unit 1)
-    (in_bom yes) (on_board yes)
-    (property "Reference" "R101" (id 0) (at 142.24 95.25 90))
-    (property "Value" "100K/1%" (id 1) (at 152.4 95.25 90))
-    (property "Footprint" "Resistor_SMD:R_0402_1005Metric" (id 2) (at 146.05 98.298 90)
-      (effects (font (size 1.27 1.27)) hide)
-    )
-    (property "Datasheet" "~" (id 3) (at 146.05 96.52 0)
-      (effects (font (size 1.27 1.27)) hide)
-    )
-    (pin "1")
-    (pin "2")
-  )
   (symbol (lib_id "Device:C") (at 97.79 73.66 90) (mirror x) (unit 1)
