File: hardware/main_pcb/pcb.kicad_pcb (KiCad board)
At the start: 2 copper layers, 0 parts

Commit message: - Initial PCB layout
Parts:
- added C1: 100nF, Capacitor_SMD:C_0402_1005Metric, B.Cu at (94.4, 71.8)
- added C10: 1uF, Capacitor_SMD:C_0402_1005Metric, B.Cu at (83.6, 72.8)
- added C100: 2.2uF, Capacitor_SMD:C_0603_1608Metric, F.Cu at (46.9, 37.0)
- added C101: 10uF, Capacitor_SMD:C_0603_1608Metric, F.Cu at (48.5, 37.5)
- added C102: 10uF, Capacitor_SMD:C_0603_1608Metric, F.Cu at (50.0, 37.5)
- added C103: 1uF, Capacitor_SMD:C_0402_1005Metric, F.Cu at (46.7, 34.9)
- added C104: 10uF, Capacitor_SMD:C_0603_1608Metric, F.Cu at (46.1, 33.5)
- added C105: 10uF, Capacitor_SMD:C_0603_1608Metric, F.Cu at (50.1, 31.1)
- added C106: 10uF, Capacitor_SMD:C_0603_1608Metric, F.Cu at (52.5, 36.8)
- added C107: 10uF, Capacitor_SMD:C_0603_1608Metric, F.Cu at (48.9, 28.0)
- added C11: 100nF, Capacitor_SMD:C_0402_1005Metric, B.Cu at (89.9, 75.7)
- added C12: 18pF, Capacitor_SMD:C_0402_1005Metric, B.Cu at (96.4, 66.7)
- added C13: 18pF, Capacitor_SMD:C_0402_1005Metric, B.Cu at (96.4, 71.8)
- added C14: 100nF, Capacitor_SMD:C_0402_1005Metric, B.Cu at (78.6, 76.0)
- added C2: 100nF, Capacitor_SMD:C_0402_1005Metric, B.Cu at (83.6, 69.8)
- added C200: 100nF, Capacitor_SMD:C_0805_2012Metric, B.Cu at (59.1, 32.5)
- added C201: 2.2uF, Capacitor_SMD:C_0603_1608Metric, B.Cu at (66.5, 32.4)
- added C3: 100nF, Capacitor_SMD:C_0402_1005Metric, B.Cu at (94.4, 70.8)
- added C300: 18pF, Capacitor_SMD:C_0402_1005Metric, B.Cu at (92.4, 65.0)
- added C301: 47uF, Capacitor_SMD:C_0805_2012Metric, F.Cu at (55.8, 34.4)
- added C302: 100nF, Capacitor_SMD:C_0402_1005Metric, B.Cu at (48.5, 41.0)
- added C4: 100nF, Capacitor_SMD:C_0402_1005Metric, B.Cu at (89.9, 65.0)
- added C5: 100nF, Capacitor_SMD:C_0402_1005Metric, B.Cu at (86.3, 65.0)
- added C500: 100nF, Capacitor_SMD:C_0402_1005Metric, B.Cu at (112.9, 59.1)
- added C501: 10uF, Capacitor_SMD:C_0603_1608Metric, F.Cu at (67.8, 36.0)
- added C502: 1uF, Capacitor_SMD:C_0402_1005Metric, B.Cu at (87.9, 62.8)
- added C503: 220pF, Capacitor_SMD:C_0603_1608Metric, B.Cu at (62.5, 43.9)
- added C504: 22uF/50V, Capacitor_SMD:C_1206_3216Metric, F.Cu at (56.1, 38.5)
- added C506: 4.7uF/50V, Capacitor_SMD:C_0805_2012Metric, F.Cu at (59.6, 40.7)
- added C507: 1uF/50V, Capacitor_SMD:C_0805_2012Metric, B.Cu at (134.5, 54.6)
- added C508: 1uF/50V, Capacitor_SMD:C_0805_2012Metric, B.Cu at (128.5, 54.6)
- added C509: 1uF/50V, Capacitor_SMD:C_0805_2012Metric, B.Cu at (122.8, 54.6)
- added C510: 1uF/50V, Capacitor_SMD:C_0805_2012Metric, B.Cu at (117.0, 54.6)
- added C511: 4.7uF/50V, Capacitor_SMD:C_0805_2012Metric, B.Cu at (117.0, 61.9)
- added C512: 4.7uF/50V, Capacitor_SMD:C_0805_2012Metric, B.Cu at (122.8, 61.9)
- added C513: 4.7uF/50V, Capacitor_SMD:C_0805_2012Metric, B.Cu at (128.5, 61.9)
- added C514: 4.7uF/50V, Capacitor_SMD:C_0805_2012Metric, B.Cu at (134.5, 61.9)
- added C515: 100nF, Capacitor_SMD:C_0402_1005Metric, B.Cu at (114.8, 82.5)
- added C6: 100nF, Capacitor_SMD:C_0402_1005Metric, B.Cu at (83.6, 70.8)
- added C7: 100nF, Capacitor_SMD:C_0402_1005Metric, B.Cu at (83.6, 73.8)
- added C8: 1uF, Capacitor_SMD:C_0402_1005Metric, B.Cu at (83.6, 71.8)
- added C9: 100nF, Capacitor_SMD:C_0402_1005Metric, B.Cu at (86.3, 75.7)
- added D501: MBR0530, Diode_SMD:D_SOD-123, F.Cu at (60.0, 37.1)
- added J1: USB_AB_Micro, Connector_USB:USB_Micro-AB_Molex_47590-0001, B.Cu at (63.5, 26.4)
- added J300: MICRO_SD(TFC-WPAPR-08), footprints:TFC-WPAPR-08, B.Cu at (49.6, 31.6)
- added J400: Conn_01x03, Connector_PinHeader_1.27mm:PinHeader_1x03_P1.27mm_Vertical, F.Cu at (67.8, 38.1)
- added J401: Conn_01x03, Connector_PinHeader_1.27mm:PinHeader_1x03_P1.27mm_Vertical, F.Cu at (134.6, 26.5)
- added J402: Conn_01x03, Connector_PinHeader_1.27mm:PinHeader_1x03_P1.27mm_Vertical, F.Cu at (134.6, 38.1)
- added J500: Conn_01x24_MountingPin, Connector_FFC-FPC:Hirose_FH12-24S-0.5SH_1x24-1MP_P0.50mm_Horizontal, B.Cu at (120.6, 75.6)
- added L100: 4.7uH, Inductor_SMD:L_Vishay_IHLP-1212, F.Cu at (46.9, 30.8)
- added L101: 4.7uH, Inductor_SMD:L_Vishay_IHLP-1212, F.Cu at (52.8, 33.5)
- added L500: 47uH, Inductor_SMD:L_Vishay_IHLP-1212, F.Cu at (63.6, 35.7)
- added MCU_JTAG1: Conn_02x05_Odd_Even, Connector_PinHeader_1.27mm:PinHeader_2x05_P1.27mm_Vertical_SMD, B.Cu at (61.8, 38.1)
- added R1: 4.7K, Capacitor_SMD:C_0402_1005Metric, B.Cu at (83.8, 61.8)
- added R101: 100K/1%, Resistor_SMD:R_0402_1005Metric, F.Cu at (51.9, 38.1)
- added R117: 4.7K, Capacitor_SMD:C_0402_1005Metric, B.Cu at (94.4, 74.0)
- added R2: 4.7K, Capacitor_SMD:C_0402_1005Metric, B.Cu at (83.8, 62.9)
- added R200: 0, Resistor_SMD:R_0805_2012Metric, B.Cu at (61.2, 32.5)
- added R201: 75K, Resistor_SMD:R_0402_1005Metric, B.Cu at (46.5, 32.4)
- added R202: 47K, Resistor_SMD:R_0402_1005Metric, B.Cu at (65.2, 32.3)
- added R3: 27, Capacitor_SMD:C_0402_1005Metric, B.Cu at (81.6, 76.2)
- added R301: 33R, Resistor_SMD:R_0402_1005Metric, B.Cu at (91.3, 65.0)
- added R302: 47K, Resistor_SMD:R_0402_1005Metric, B.Cu at (51.9, 41.1)
- added R305: 47K, Resistor_SMD:R_0402_1005Metric, B.Cu at (44.1, 41.0)
- added R306: 47K, Resistor_SMD:R_0402_1005Metric, B.Cu at (45.3, 41.0)
- added R307: 47K, Resistor_SMD:R_0402_1005Metric, F.Cu at (57.4, 35.1)
- added R308: 47K, Resistor_SMD:R_0402_1005Metric, B.Cu at (50.8, 41.1)
- added R4: 27, Capacitor_SMD:C_0402_1005Metric, B.Cu at (81.6, 77.2)
- added R5: 1k, Capacitor_SMD:C_0402_1005Metric, B.Cu at (78.1, 64.5)
- added R500: 100K/1%, Resistor_SMD:R_0402_1005Metric, B.Cu at (106.1, 59.4)
- added R501: 100K/1%, Resistor_SMD:R_0402_1005Metric, B.Cu at (106.1, 58.2)
- added R502: 100K/1%, Resistor_SMD:R_0402_1005Metric, B.Cu at (106.1, 57.1)
- added R503: 100K/1%, Resistor_SMD:R_0402_1005Metric, B.Cu at (106.1, 56.0)
- added R504: 10K, Resistor_SMD:R_0402_1005Metric, B.Cu at (87.9, 65.0)
- added R505: 47K, Resistor_SMD:R_0402_1005Metric, B.Cu at (64.1, 43.4)
- added R506: 4.7K, Resistor_SMD:R_0402_1005Metric, B.Cu at (65.7, 43.4)
- added R507: 330K/1%, Resistor_SMD:R_0402_1005Metric, B.Cu at (68.4, 43.4)
- added R508: 18K/1%, Resistor_SMD:R_0402_1005Metric, B.Cu at (67.0, 43.4)
- added R509: 220K/1%, Resistor_SMD:R_0402_1005Metric, B.Cu at (119.7, 60.5)
- added R510: 18K/1%, Resistor_SMD:R_0402_1005Metric, B.Cu at (119.7, 58.2)
- added R511: 220K/1%, Resistor_SMD:R_0402_1005Metric, B.Cu at (125.5, 60.5)
- added R512: 18K/1%, Resistor_SMD:R_0402_1005Metric, B.Cu at (125.5, 58.2)
- added R513: 220K/1%, Resistor_SMD:R_0402_1005Metric, B.Cu at (131.2, 60.5)
- added R514: 18K/1%, Resistor_SMD:R_0402_1005Metric, B.Cu at (131.2, 58.2)
- added R515: 220K/1%, Resistor_SMD:R_0402_1005Metric, B.Cu at (137.1, 60.5)
- added R516: 18K/1%, Resistor_SMD:R_0402_1005Metric, B.Cu at (137.1, 58.2)
- added R517: 33, Resistor_SMD:R_0402_1005Metric, B.Cu at (114.8, 76.3)
- added R6: DNP, Capacitor_SMD:C_0402_1005Metric, B.Cu at (76.9, 64.5)
- added R7: 1k, Capacitor_SMD:C_0402_1005Metric, B.Cu at (94.4, 69.8)
- added R8: 4.7K, Capacitor_SMD:C_0402_1005Metric, B.Cu at (94.4, 73.0)
- added RN500: 33R, Resistor_SMD:R_Array_Convex_4x0402, B.Cu at (114.8, 73.9)
- added RN501: 33R, Resistor_SMD:R_Array_Convex_4x0402, B.Cu at (114.8, 78.1)
- added RN502: 33R, Resistor_SMD:R_Array_Convex_4x0402, B.Cu at (114.8, 80.7)
- added SW1: SKQG, Button_Switch_SMD:SW_SPST_SKQG_WithStem, B.Cu at (134.9, 33.5)
- added SW400: SKQG, Button_Switch_SMD:SW_SPST_SKQG_WithStem, F.Cu at (45.5, 59.1)
- added SW401: SKQG, Button_Switch_SMD:SW_SPST_SKQG_WithStem, F.Cu at (45.5, 75.2)
- added U1: RP2040, Package_DFN_QFN:QFN-56-1EP_7x7mm_P0.4mm_EP5.6x5.6mm_ThermalVias, B.Cu at (88.9, 70.3)
- added U100: ADP5360, footprints:WLCSP-32_6x6_2.56x2.56mm, F.Cu at (49.3, 34.3)
- added U2: W25Q128JVS, Package_SO:SOIC-8_5.23x5.23mm_P1.27mm, B.Cu at (79.5, 70.5)
- added U200: NX5P2090, footprints:WLCSP-9_3x3_1.36x1.36mm, B.Cu at (68.4, 32.2)
- added U201: NX18P3001, footprints:WLCSP-12_3x4_1.36x1.66mm, B.Cu at (63.5, 32.1)
- added U300: NX3P1108UK, Package_CSP:WLCSP-4-X1-WLB0909-4_0.89x0.89mm_P0.5mm, F.Cu at (58.4, 32.6)
- added U500: DS4424, Package_DFN_QFN:DFN-14-1EP_3x3mm_P0.4mm_EP1.78x2.35mm, B.Cu at (109.5, 58.4)
- added U501: NX3P1108UK, Package_CSP:WLCSP-4-X1-WLB0909-4_0.89x0.89mm_P0.5mm, B.Cu at (121.7, 49.5)
- added U502: LT1615, Package_TO_SOT_SMD:TSOT-23-5, F.Cu at (63.6, 39.4)
- added U503: MIC5233YM5, Package_TO_SOT_SMD:SOT-23-5, B.Cu at (117.0, 58.2)
- added U504: MIC5233YM5, Package_TO_SOT_SMD:SOT-23-5, B.Cu at (122.8, 58.2)
- added U505: MIC5233YM5, Package_TO_SOT_SMD:SOT-23-5, B.Cu at (128.6, 58.2)
- added U506: MIC5233YM5, Package_TO_SOT_SMD:SOT-23-5, B.Cu at (134.6, 58.2)
- added Y1: 24MHz, Oscillator:Oscillator_SMD_Abracon_ASE-4Pin_3.2x2.5mm, B.Cu at (97.2, 69.2)
Other:
- board outline added: 100 x 60 mm
- copper layers 2 -> 4

Commit message: - PCB rev 0p1 draft
Parts:
- removed R101: 100K/1%, Resistor_SMD:R_0402_1005Metric
- R307, U300: moved to B.Cu
- moved U501 69.6 mm to (52.4, 43.2)
- moved R201 20.5 mm to (66.9, 34.3), turned to -90 degrees
- moved U300 13.5 mm to (49.9, 43.2)
- moved C301 12.1 mm to (44.0, 37.3)
- moved R307 9.80 mm to (49.6, 41.1), turned to 90 degrees
- moved C14 8.63 mm to (76.0, 67.7), turned to 90 degrees
- moved C501 7.00 mm to (62.5, 40.6), turned to 180 degrees
- moved R5 5.70 mm to (78.1, 58.8)
- moved R6 5.70 mm to (76.9, 58.8)
- moved U2 5.70 mm to (79.5, 64.8)
- moved U505 5.50 mm to (123.0, 58.2)
- moved C500 5.50 mm to (107.4, 59.1)
- moved C507 5.50 mm to (129.0, 54.6)
- moved C508 5.50 mm to (123.0, 54.6)
- moved C509 5.50 mm to (117.3, 54.6)
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Connections:
- J500 pad 12: /cpu/GPIO11 -> /cpu/GPIO15
- R517 pad 2: /cpu/GPIO14 -> /cpu/GPIO16
- RN500 pad 5: /cpu/GPIO12 -> /cpu/GPIO14
- RN500 pad 7: /cpu/GPIO16 -> /cpu/GPIO12
- RN500 pad 8: /cpu/GPIO15 -> /cpu/GPIO11
- RN501 pad 5: /cpu/GPIO21 -> /cpu/GPIO20
- RN501 pad 6: /cpu/GPIO22 -> /cpu/GPIO19
- RN501 pad 7: /cpu/GPIO23 -> /cpu/GPIO18
- RN501 pad 8: /cpu/GPIO24 -> /cpu/GPIO17
- RN502 pad 5: /cpu/GPIO17 -> /cpu/GPIO24
- RN502 pad 6: /cpu/GPIO18 -> /cpu/GPIO23
- RN502 pad 7: /cpu/GPIO19 -> /cpu/GPIO22
- RN502 pad 8: /cpu/GPIO20 -> /cpu/GPIO21
Routing:
- net +3V3: track 0.00 -> 333.1 mm, vias 0 -> 16
- net +BATT: track 0.00 -> 200.7 mm, vias 0 -> 3
- net VEE: track 0.00 -> 162.9 mm, vias 0 -> 3
- net /cpu/GPIO27_ADC1: track 0.00 -> 162.4 mm, vias 0 -> 1
- net /cpu/GPIO26_ADC0: track 0.00 -> 161.5 mm, vias 0 -> 1
- net +3V3_LCD: track 0.00 -> 149.7 mm, vias 0 -> 2
- net BAT_NTC: track 0.00 -> 98.3 mm, vias 0 -> 1
- net /cpu/GPIO0: track 0.00 -> 87.3 mm, vias 0 -> 4
- net /cpu/GPIO1: track 0.00 -> 86.6 mm, vias 0 -> 4
- net /cpu/SWD: track 0.00 -> 83.1 mm, vias 0 -> 4
- net /cpu/~USB_BOOT: track 0.00 -> 80.3 mm, vias 0 -> 4
- net /cpu/SWCLK: track 0.00 -> 79.4 mm, vias 0 -> 4
- net /cpu/GPIO2: track 0.00 -> 74.1 mm, vias 0 -> 1
- net /cpu/GPIO6: track 0.00 -> 68.2 mm
- net /cpu/GPIO25: track 0.00 -> 66.9 mm, vias 0 -> 2
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- added copper zone on B.Cu, net GND
- added copper zone on F.Cu, net GND
Other:
- copper layers 4 -> 2
- board text added: "Copyright 2021 Wenting Zhang"
- board text added: "P"
- board text added: "READER"
- board text added: "Rev 0.1 PROTOTYPE"
- board text added: "VREF SWD GND SWC GND NC NC NC NC NC"

Commit message: - harware rev 0.1 freeze
Parts:
- moved C302 1.03 mm to (48.5, 42.1)
- moved R305 1.02 mm to (44.1, 42.0)
- moved R306 1.02 mm to (45.3, 42.0)
- moved R302 0.93 mm to (51.9, 42.1)
- moved R307 0.93 mm to (49.6, 42.1)
- moved R308 0.93 mm to (50.8, 42.1)
- moved U501 0.88 mm to (52.4, 44.0)
- moved U300 0.88 mm to (49.9, 44.0)
- moved J300 0.85 mm to (49.6, 32.4)
Routing:
- net /cpu/GPIO27_ADC1: track 162.4 -> 163.7 mm
- net /cpu/GPIO4: track 59.6 -> 58.4 mm
- net /cpu/GPIO9: track 65.7 -> 66.7 mm
- net Net-(C300-Pad1): track 65.4 -> 66.3 mm
- net GND: track 63.2 -> 62.4 mm, vias 147 -> 149
- net +3V3: track 333.1 -> 333.9 mm
- net +VSD: track 18.6 -> 19.4 mm
- net /cpu/GPIO26_ADC0: track 161.5 -> 162.2 mm
- net /cpu/GPIO6: track 68.2 -> 67.7 mm
