File: hardware/front_pcb/front_pcb.kicad_pcb (KiCad board)
At the start: 2 copper layers, 120 x 160 mm, 13 parts, among them J1 Conn_01x06, J2 Conn_01x06, J3 Conn_01x03, J4 Conn_01x03, J5 Conn_01x03, SW1 EVQPUJ02K, SW2 EVQPUJ02K, U1 MPR121QR2

Commit message: - PCB rev 0p1 draft
Parts:
- moved TH1 60.9 mm to (129.7, 40.2), turned to -90 degrees
- moved R1 1.16 mm to (44.4, 33.4), turned to -90 degrees
- moved C2 0.10 mm to (46.9, 36.0)
Routing:
- net Net-(J2-Pad6): track 0.00 -> 184.8 mm, vias 0 -> 1
- net Net-(J2-Pad5): track 0.00 -> 177.5 mm, vias 0 -> 1
- net Net-(J2-Pad4): track 0.00 -> 170.9 mm, vias 0 -> 1
- net GND: track 0.00 -> 165.1 mm, vias 0 -> 8
- net Net-(J2-Pad3): track 0.00 -> 164.5 mm, vias 0 -> 1
- net Net-(J2-Pad2): track 0.00 -> 158.8 mm, vias 0 -> 1
- net Net-(J2-Pad1): track 0.00 -> 152.9 mm, vias 0 -> 1
- net Net-(J1-Pad6): track 0.00 -> 108.8 mm, vias 0 -> 1
- net Net-(J1-Pad5): track 0.00 -> 100.5 mm, vias 0 -> 1
- net +3V3: track 0.00 -> 93.9 mm, vias 0 -> 2
- net Net-(J1-Pad4): track 0.00 -> 92.0 mm, vias 0 -> 1
- net /KEY2: track 0.00 -> 87.5 mm
- net Net-(J1-Pad3): track 0.00 -> 81.9 mm, vias 0 -> 1
- net Net-(J1-Pad2): track 0.00 -> 74.1 mm, vias 0 -> 1
- net /KEY1: track 0.00 -> 71.3 mm
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- added copper zone on B.Cu, net GND
- added copper zone on F.Cu, net GND
Other:
- board text added: "P"
- board text added: "READER"
- board text removed: "Preader"

Commit message: - harware rev 0.1 freeze
Changed lines of the file:
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@@
       (viasonmask false)
       (mode 1)
-      (useauxorigin false)
+      (useauxorigin true)
       (hpglpennumber 1)
       (hpglpenspeed 20)
@@
       (outputformat 1)
       (mirror false)
-      (drillshape 1)
+      (drillshape 0)
       (scaleselection 1)
-      (outputdirectory "")
+      (outputdirectory "gerber/")
     )
   )
@@
     (property "Sheetname" "")
     (attr smd)
-    (fp_text reference "J5" (at 0 2.965) (layer "B.SilkS")
+    (fp_text reference "J5" (at -4.6 0.1) (layer "B.SilkS")
       (effects (font (size 1 1) (thickness 0.15)) (justify mirror))
     )
@@
     (property "Sheetname" "")
     (attr smd)
-    (fp_text reference "SW1" (at 0 4.5 90) (layer "B.SilkS")
+    (fp_text reference "SW1" (at 0 -3.5 90) (layer "B.SilkS")
       (effects (font (size 1 1) (thickness 0.15)) (justify mirror))
     )
@@
     (property "Sheetname" "")
     (attr smd)
-    (fp_text reference "TH1" (at 0 1.43 -90) (layer "B.SilkS")
+    (fp_text reference "TH1" (at -2.3 -0.6 180) (layer "B.SilkS")
       (effects (font (size 1 1) (thickness 0.15)) (justify mirror))
     )
@@
     (property "Sheetname" "")
     (attr through_hole)
-    (fp_text reference "BT1" (at 4.88 9.42 180) (layer "B.SilkS")
+    (fp_text reference "BT1" (at 0.4 7.1 180) (layer "B.SilkS")
       (effects (font (size 1 1) (thickness 0.15)) (justify mirror))
     )
@@
       (effects (font (size 1 1) (thickness 0.15)) (justify mirror))
     )
-    (fp_text user "-" (at 60.27 0.06) (layer "B.SilkS")
-      (effects (font (size 1 1) (thickness 0.15)) (justify mirror))
-    )
-    (fp_text user "+" (at 1.5 0.06) (layer "B.SilkS")
+    (fp_text user "-" (at 60.4 4.5) (layer "B.SilkS")
+      (effects (font (size 1 1) (thickness 0.15)) (justify mirror))
+    )
+    (fp_text user "+" (at 1.4 4.3) (layer "B.SilkS")
       (effects (font (size 1 1) (thickness 0.15)) (justify mirror))
     )
@@
     (property "Sheetname" "")
     (attr smd)
-    (fp_text reference "J3" (at 0 2.965) (layer "B.SilkS")
+    (fp_text reference "J3" (at 2.2 1.3) (layer "B.SilkS")
       (effects (font (size 1 1) (thickness 0.15)) (justify mirror))
     )
@@
     (property "Sheetname" "")
     (attr smd)
-    (fp_text reference "U1" (at 0 2.8 270) (layer "B.SilkS")
+    (fp_text reference "U1" (at 1.2 3 270) (layer "B.SilkS")
       (effects (font (size 1 1) (thickness 0.15)) (justify mirror))
     )
@@
     (property "Sheetname" "")
     (attr smd)
-    (fp_text reference "J4" (at 0 2.965) (layer "B.SilkS")
+    (fp_text reference "J4" (at -4.7 -0.1) (layer "B.SilkS")
       (effects (font (size 1 1) (thickness 0.15)) (justify mirror))
     )
@@
     (property "Sheetname" "")
     (attr smd)
-    (fp_text reference "SW2" (at 0 4.5 90) (layer "B.SilkS")
+    (fp_text reference "SW2" (at 0.2 -3.4 90) (layer "B.SilkS")
       (effects (font (size 1 1) (thickness 0.15)) (justify mirror))
     )
@@
   (gr_line (start 52.5 47.5) (end 52.5 172.5) (layer "Edge.Cuts") (width 0.05))
   (gr_line (start 147.5 47.5) (end 52.5 47.5) (layer "Edge.Cuts") (width 0.05))
-  (gr_text "P" (at 86 36.5) (layer "F.Cu")
-    (effects (font (size 6 5) (thickness 0.8)))
-  )
-  (gr_text "READER" (at 102.5 37) (layer "F.Cu")
+  (gr_text "P" (at 86 37.3) (layer "F.Cu")
+    (effects (font (size 4 5) (thickness 0.8)))
+  )
+  (gr_text "READER" (at 102.5 36.9) (layer "F.Cu")
     (effects (font (size 5 5) (thickness 0.8)))
   )
-  (gr_text "READER" (at 102.5 37) (layer "F.Paste")
+  (gr_text "READER" (at 102.5 36.9) (layer "F.Paste")
     (effects (font (size 5 5) (thickness 0.8)))
   )
-  (gr_text "P" (at 86 36.5) (layer "F.Paste")
-    (effects (font (size 6 5) (thickness 0.8)))
-  )
-  (gr_text "READER" (at 102.5 37) (layer "F.Mask")
+  (gr_text "P" (at 86 37.3) (layer "F.Paste")
+    (effects (font (size 4 5) (thickness 0.8)))
+  )
+  (gr_text "READER" (at 102.5 36.9) (layer "F.Mask")
     (effects (font (size 5 5) (thickness 0.8)))
   )
-  (gr_text "P" (at 86 36.5) (layer "F.Mask")
-    (effects (font (size 6 5) (thickness 0.8)))
+  (gr_text "P" (at 86 37.3) (layer "F.Mask")
+    (effects (font (size 4 5) (thickness 0.8)))
   )
   (via (at 47.8125 37.6875) (size 0.7) (drill 0.3) (layers "F.Cu" "B.Cu") (net 1))
